File: kicad/stereo-camera-board.sch (KiCad schematic (older format))
At the start: 121 parts, among them IC1 ZLDO1117G33TA, IC2 MCP1700T-2502E/TT, IC3 SN74LVC1T45DCKR, IC4 SN74LVC1T45DCKR, IC5 MT9V032, J4 DIGILENT-JTAG, U1 ATXMEGA256A3-AU

Commit message: Generated pdf version of schematic
Parts:
- +2V5, +3V3, +3V?, +5V, +?, CMT821, EXT_SENSOR, FRAME, GND, GND1, GND10, GND11, GND12, GND13, GND14, GND15, GND16, GND17, GND18, GND19, GND2, GND20, GND3, GND4, GND5, GND6, GND7, GND8, GND9, J1, JP1, JP2, JP3, JP4, LD1, LD2, LD3, PDIJTAG: value (none) -> ~
- gave numbers to parts that had none: 1
Connections:
- wire segments 434 -> 428

Commit message: Added line from capacitor bank to +3.3
Parts:
- added +3V?: ~, symbol P+_+3V3
- added FB1: MPZ1608B471A, symbol FB_FERRITE
Connections:
- wire segments 428 -> 555

Commit message: Added led components fixed power lines and misc pieces
Parts:
- removed +2V5 (x2): ~, symbol P+_+2V5
- removed +3V3 (x14), +3V? (x2), +?: ~, symbol P+_+3V3
- removed +5V (x2): ~, symbol P+_+5V
- removed GND, GND1, GND10, GND11, GND12, GND13, GND14 (x2), GND15, GND16, GND17, GND18, GND19, GND2, GND20, GND3, GND4, GND5, GND6, GND7, GND8, GND9: ~, symbol SUPPLY_GND
- removed JP4: ~, symbol JP_JP3Q
- removed LD1, LD2, LD3: ~, symbol LD_LED
- added BLUE_LED?: LED_B, symbol LED_B
- added GREEN_LED?: LED_G, symbol LED_G
- added JP?: JP2Q, jumper-JP2Q, symbol JP2Q
- added JP?: JP_JP1Q, jumper-JP1, symbol JP_JP1Q
- added P+? (x2): +5V, symbol +5V
- added P+? (x17): +3.3V, symbol +3.3V
- added P+? (x2): +2.5V, symbol +2.5V
- added RED_LED?: LED_R, symbol LED_R
- added SUPPLY? (x22): GND, symbol GND

Commit message: Fixed ferrite component added custom.lib for all library modifications
Parts:
- removed +3V3: ~, symbol P+_+3V3
- removed EXT_SENSOR: ~, symbol JP_JP4E
- removed FB1 (x2): MPZ1608B471A, symbol FB_FERRITE
- removed FRAME (x2): ~, symbol FRAME_FRAME_B_L
- removed PDIJTAG: ~, symbol JP_PINHD-2X3
- removed SATA_PRIMARY, SATA_SLAVE_EXT: 67800-5005, symbol J_SATA7
- added EXT_SENSOR1: ~, symbol JP_JP4E
- added FB1, FB2: FERRITE, dan-rcl-0402, symbol FERRITE
- added FRAME1, FRAME2: ~, symbol FRAME_FRAME_B_L
- added P+22: +3.3V, symbol +3.3V
- added PDIJTAG1: ~, symbol JP_PINHD-2X3
- added SATA_PRIMARY1, SATA_SLAVE_EXT1: 67800-5005, symbol J_SATA7
- gave numbers to parts that had none: 55
Connections:
- wire segments 555 -> 554

Commit message: Fixed annotation
Parts:
- renumbered C1 to C31
Changed lines of the file:
@@
 $EndComp
 $Comp
-L C_C C1
+L C_C C31
 U 1 1 51F99F60
 P 4250 3450
-F 0 "C1" V 4250 3450 30  0000 R CNN
+F 0 "C31" V 4250 3450 30  0000 R CNN
 F 1 "100nF" V 4250 3350 30  0000 C CNN
 F 2 "" H 4250 3450 30  0001 C CNN

Commit message: Moved MPU-9150 to custom.lib Added no-connect pins to MPU-9150
Parts:
- removed U$1: MPU-9150, symbol mpu9150_MPU-9150
- added C?: 2.2nf, symbol C_C
- added MPU91501: MPU-9150, symbol MPU-9150
Connections:
- wire segments 554 -> 429

Commit message: Added annotation
Parts:
- gave numbers to parts that had none: 1
Changed lines of the file:
@@
 LIBS:led
 LIBS:custom
+LIBS:stereo-camera-board-cache
 EELAYER 24 0
 EELAYER END
@@
 $EndComp
 $Comp
-L C_C C?
+L C_C C32
 U 1 1 520FE1CE
 P 7350 3200
-F 0 "C?" V 7350 3200 30  0000 C CNN
+F 0 "C32" V 7350 3200 30  0000 C CNN
 F 1 "2.2nf" V 7350 3100 30  0000 C CNN
 F 2 "" H 7350 3200 30  0001 C CNN

Commit message: Connected pixclk
Connections:
- wire segments 429 -> 434
- no-connect marks 0 -> 8
Changed lines of the file:
@@
 L JP_PINHD-2X3 PDIJTAG1
 U 1 1 520F18B7
-P 4100 5850
-F 0 "PDIJTAG1" H 3950 5950 30  0000 C CNN
-F 1 "~" H 4100 5850 30  0001 C CNN
-F 2 "" H 4100 5850 30  0001 C CNN
-F 3 "" H 4100 5850 30  0001 C CNN
-	1    4100 5850
+P 4100 5950
+F 0 "PDIJTAG1" H 3950 6050 30  0000 C CNN
+F 1 "~" H 4100 5950 30  0001 C CNN
+F 2 "" H 4100 5950 30  0001 C CNN
+F 3 "" H 4100 5950 30  0001 C CNN
+	1    4100 5950
 	1    0    0    -1
 $EndComp
@@
 L R_R R8
 U 1 1 520F18D3
-P 3400 5750
-F 0 "R8" H 3500 5750 30  0000 C CNN
-F 1 "1K" H 3350 5750 30  0000 C CNN
-F 2 "" H 3400 5750 30  0001 C CNN
-F 3 "" H 3400 5750 30  0001 C CNN
-	1    3400 5750
+P 3400 5850
+F 0 "R8" H 3500 5850 30  0000 C CNN
+F 1 "1K" H 3350 5850 30  0000 C CNN
+F 2 "" H 3400 5850 30  0001 C CNN
+F 3 "" H 3400 5850 30  0001 C CNN
+	1    3400 5850
 	0    -1   -1   0
 $EndComp
@@
 L R_R R9
 U 1 1 520F18D2
-P 3450 5750
-F 0 "R9" H 3550 5750 30  0000 C CNN
-F 1 "1K" H 3400 5750 30  0000 C CNN
-F 2 "" H 3450 5750 30  0001 C CNN
-F 3 "" H 3450 5750 30  0001 C CNN
-	1    3450 5750
+P 3450 5850
+F 0 "R9" H 3550 5850 30  0000 C CNN
+F 1 "1K" H 3400 5850 30  0000 C CNN
+F 2 "" H 3450 5850 30  0001 C CNN
+F 3 "" H 3450 5850 30  0001 C CNN
+	1    3450 5850
 	0    -1   -1   0
 $EndComp
@@
 L C_C C27
 U 1 1 51F99F85
-P 4200 4250
-F 0 "C27" V 4200 4250 30  0000 C CNN
-F 1 "100nF" V 4200 4200 30  0000 C CNN
-F 2 "" H 4200 4250 30  0001 C CNN
-F 3 "" H 4200 4250 30  0001 C CNN
-	1    4200 4250
+P 4325 3950
+F 0 "C27" V 4325 3950 30  0000 C CNN
+F 1 "100nF" V 4325 3900 30  0000 C CNN
+F 2 "" H 4325 3950 30  0001 C CNN
+F 3 "" H 4325 3950 30  0001 C CNN
+	1    4325 3950
 	1    0    0    -1
 $EndComp
@@
 L C_C C10
 U 1 1 51F99F97
-P 3750 5800
-F 0 "C10" V 3750 5800 30  0000 C CNN
-F 1 "100nF" V 3750 5750 30  0000 C CNN
-F 2 "" H 3750 5800 30  0001 C CNN
-F 3 "" H 3750 5800 30  0001 C CNN
-	1    3750 5800
+P 3750 5900
+F 0 "C10" V 3750 5900 30  0000 C CNN
+F 1 "100nF" V 3750 5850 30  0000 C CNN
+F 2 "" H 3750 5900 30  0001 C CNN
+F 3 "" H 3750 5900 30  0001 C CNN
+	1    3750 5900
 	1    0    0    -1
 $EndComp
@@
 	3550 3650 3400 3650
 Wire Wire Line
-	3900 5650 5000 5650
-Wire Wire Line
-	3900 5800 3900 5650
+	5000 5750 3900 5750
+Wire Wire Line
+	3900 5900 3900 5750
 Wire Wire Line
 	4000 4600 4000 2900
@@
 	5700 4450 5700 4350
 Wire Wire Line
-	3900 6100 3900 5900
-Wire Wire Line
-	4550 6100 3900 6100
-Wire Wire Line
-	4550 5700 4550 6100
-Wire Wire Line
-	5050 5700 4550 5700
-Wire Wire Line
-	5050 3450 5050 5700
+	3900 6200 3900 6000
+Wire Wire Line
+	4550 6200 3900 6200
+Wire Wire Line
+	4550 5800 4550 6200
+Wire Wire Line
+	5050 5800 4550 5800
+Wire Wire Line
+	5050 3450 5050 5800
 Wire Wire Line
 	5150 3450 5150 3500
@@
 	5050 3450 5150 3450
 Wire Wire Line
-	5000 5650 5000 3400
+	5000 3400 5000 5750
 Wire Wire Line
 	5200 3400 5200 3500
@@
 	7400 5150 7400 5350
 Wire Wire Line
-	3450 5650 3450 5150
+	3450 5150 3450 5750
 Connection ~ 3450 5150
 Wire Wire Line
-	3400 5650 3400 5100
+	3400 5100 3400 5750
 Connection ~ 3400 5100
 Wire Wire Line
-	3450 5850 3450 5900
-Wire Wire Line
-	3400 5900 3600 5900
-Wire Wire Line
-	3400 5850 3400 5900
-Connection ~ 3450 5900
+	3450 5950 3450 6000
+Wire Wire Line
+	3400 6000 3600 6000
+Wire Wire Line
+	3400 5950 3400 6000
+Connection ~ 3450 6000
 Wire Wire Line
 	7650 4000 8100 4000
@@
 	3050 2450 5350 2450
 Wire Wire Line
-	4350 5800 4250 5800
-Wire Wire Line
-	4250 5900 4450 5900
-Wire Wire Line
-	3900 5900 3950 5900
-Wire Wire Line
-	3950 5800 3900 5800
+	4350 5900 4250 5900
+Wire Wire Line
+	4250 6000 4450 6000
+Wire Wire Line
+	3900 6000 3950 6000
+Wire Wire Line
+	3950 5900 3900 5900
 Connection ~ 4250 3350
 Wire Wire Line
@@
 L GND SUPPLY10
 U 1 1 520EEFC7
-P 4450 5950
-F 0 "SUPPLY10" H 4450 5950 30  0001 L BNN
-F 1 "GND" H 4402 5870 30  0000 L BNN
-F 2 "" H 4450 5950 60  0000 C CNN
-F 3 "" H 4450 5950 60  0000 C CNN
-	1    4450 5950
+P 4450 6050
+F 0 "SUPPLY10" H 4450 6050 30  0001 L BNN
+F 1 "GND" H 4402 5970 30  0000 L BNN
+F 2 "" H 4450 6050 60  0000 C CNN
+F 3 "" H 4450 6050 60  0000 C CNN
+	1    4450 6050
 	1    0    0    -1
 $EndComp
@@
 L +3.3V P+11
 U 1 1 520EEFD6
-P 4350 5750
-F 0 "P+11" V 4350 5750 50  0001 L BNN
-F 1 "+3.3V" V 4400 5750 30  0000 L BNN
-F 2 "" H 4350 5750 60  0000 C CNN
-F 3 "" H 4350 5750 60  0000 C CNN
-	1    4350 5750
+P 4350 5850
+F 0 "P+11" V 4350 5850 50  0001 L BNN
+F 1 "+3.3V" V 4400 5850 30  0000 L BNN
+F 2 "" H 4350 5850 60  0000 C CNN
+F 3 "" H 4350 5850 60  0000 C CNN
+	1    4350 5850
 	1    0    0    -1
 $EndComp
@@
 L GND SUPPLY6
 U 1 1 520EEFE5
-P 3750 5950
-F 0 "SUPPLY6" H 3750 5950 30  0001 L BNN
-F 1 "GND" H 3702 5870 30  0000 L BNN
-F 2 "" H 3750 5950 60  0000 C CNN
-F 3 "" H 3750 5950 60  0000 C CNN
-	1    3750 5950
+P 3750 6050
+F 0 "SUPPLY6" H 3750 6050 30  0001 L BNN
+F 1 "GND" H 3702 5970 30  0000 L BNN
+F 2 "" H 3750 6050 60  0000 C CNN
+F 3 "" H 3750 6050 60  0000 C CNN
+	1    3750 6050
 	1    0    0    -1
 $EndComp
@@
 L +3.3V P+7
 U 1 1 520EEFF4
-P 3600 5850
-F 0 "P+7" V 3600 5850 50  0001 L BNN
-F 1 "+3.3V" V 3650 5850 30  0000 L BNN
-F 2 "" H 3600 5850 60  0000 C CNN
-F 3 "" H 3600 5850 60  0000 C CNN
-	1    3600 5850
+P 3600 5950
+F 0 "P+7" V 3600 5950 50  0001 L BNN
+F 1 "+3.3V" V 3650 5950 30  0000 L BNN
+F 2 "" H 3600 5950 60  0000 C CNN
+F 3 "" H 3600 5950 60  0000 C CNN
+	1    3600 5950
 	1    0    0    -1
 $EndComp
@@
 L GND SUPPLY8
 U 1 1 520EF012
-P 4200 4400
-F 0 "SUPPLY8" H 4200 4400 30  0001 L BNN
-F 1 "GND" H 4152 4320 30  0000 L BNN
-F 2 "" H 4200 4400 60  0000 C CNN
-F 3 "" H 4200 4400 60  0000 C CNN
-	1    4200 4400
+P 4325 4100
+F 0 "SUPPLY8" H 4325 4100 30  0001 L BNN
+F 1 "GND" H 4277 4020 30  0000 L BNN
+F 2 "" H 4325 4100 60  0000 C CNN
+F 3 "" H 4325 4100 60  0000 C CNN
+	1    4325 4100
 	1    0    0    -1
 $EndComp
@@
 L +3.3V P+9
 U 1 1 520EF021
-P 4200 4150
-F 0 "P+9" V 4200 4150 50  0001 L BNN
-F 1 "+3.3V" V 4250 4150 30  0000 L BNN
-F 2 "" H 4200 4150 60  0000 C CNN
-F 3 "" H 4200 4150 60  0000 C CNN
-	1    4200 4150
+P 4325 3850
+F 0 "P+9" V 4325 3850 50  0001 L BNN
+F 1 "+3.3V" V 4375 3850 30  0000 L BNN
+F 2 "" H 4325 3850 60  0000 C CNN
+F 3 "" H 4325 3850 60  0000 C CNN
+	1    4325 3850
 	1    0    0    -1
 $EndComp
@@
 L +3.3V P+8
 U 1 1 520F1641
-P 3750 5700
-F 0 "P+8" V 3750 5700 50  0001 L BNN
-F 1 "+3.3V" V 3800 5700 30  0000 L BNN
-F 2 "" H 3750 5700 60  0000 C CNN
-F 3 "" H 3750 5700 60  0000 C CNN
-	1    3750 5700
+P 3750 5800
+F 0 "P+8" V 3750 5800 50  0001 L BNN
+F 1 "+3.3V" V 3800 5800 30  0000 L BNN
+F 2 "" H 3750 5800 60  0000 C CNN
+F 3 "" H 3750 5800 60  0000 C CNN
+	1    3750 5800
 	1    0    0    -1
 $EndComp
@@
 	7250 3200 7250 2700
 Connection ~ 7250 2700
+Connection ~ 7100 2700
+NoConn ~ 8325 4800
+NoConn ~ 8375 4800
+NoConn ~ 8425 4800
+NoConn ~ 8475 4800
+NoConn ~ 4250 5950
+NoConn ~ 3950 5950
+Connection ~ 8050 2700
+NoConn ~ 3400 3850
+NoConn ~ 3400 3900
+Connection ~ 1100 2400
+Wire Wire Line
+	5650 4500 5650 5650
+Wire Wire Line
+	5650 5650 4100 5650
+Wire Wire Line
+	4100 5650 4100 2800
+Wire Wire Line
+	4100 2800 2750 2800
+Wire Wire Line
+	2750 2800 2750 3100
 $EndSCHEMATC
