File: kicad/stereo-camera-board.sch (KiCad schematic (older format))
At the start: 125 parts, among them IC1 ZLDO1117G33TA, IC2 MCP1700T-2502E/TT, IC3 SN74LVC1T45DCKR, IC4 SN74LVC1T45DCKR, IC5 MT9V032, J4 DIGILENT-JTAG, U1 ATXMEGA256A3-AU

Commit message: Added bead to schematic
Parts:
- removed C27, C31: 100nF, symbol C_C
- removed C30: 10uF, symbol C_C
- removed P+14, P+9: +3.3V, symbol +3.3V
- removed SUPPLY13, SUPPLY8: GND, symbol GND
- added ???: BEAD, symbol BEAD
- added C27: 10uF, symbol C_CPOL
Connections:
- wire segments 434 -> 571
Other:
- moved on the sheet: FB2

Commit message: Fix no connects and connections on mpu
Parts:
- removed C11: 100nF, symbol C_C
- removed C32: 2.2nf, symbol C_C
- removed P+10, P+21: +3.3V, symbol +3.3V
- removed SUPPLY14, SUPPLY20, SUPPLY21: GND, symbol GND
- added C30: 10uF, symbol C_CPOL
- added C31: 100nF, symbol C_C
- added P+9: +3.3V, symbol +3.3V
- added SUPPLY13, SUPPLY8: GND, symbol GND
- gave numbers to parts that had none: 1
Connections:
- wire segments 571 -> 434
- no-connect marks 8 -> 9
Other:
- moved on the sheet: ??1, FB2

Commit message: Added no connect to pr0 and pr1 on xmega Downloaded correct pdf Updated schematic pdf Deleted old duplicate pdf
Parts:
- removed P+19: +3.3V, symbol +3.3V
Connections:
- net labels removed: BP, N$29
- no-connect marks 9 -> 11
Changed lines of the file:
@@
 U 1 1 520F18F3
 P 8250 2600
-F 0 "C22" V 8250 2600 30  0000 C CNN
-F 1 ".1uf" V 8250 2500 30  0000 C CNN
+F 0 "C22" V 8220 2640 30  0000 C CNN
+F 1 ".1uf" V 8180 2560 30  0000 C CNN
 F 2 "" H 8250 2600 30  0001 C CNN
 F 3 "" H 8250 2600 30  0001 C CNN
@@
 U 1 1 520F18E9
 P 8400 4300
-F 0 "EXT_SENSOR1" V 8350 4250 30  0000 C CNN
+F 0 "EXT_SENSOR1" V 8300 4250 30  0000 C CNN
 F 1 "~" H 8400 4250 30  0001 C CNN
 F 2 "" H 8400 4250 30  0001 C CNN
@@
 	-1   0    0    1
 $EndComp
-Text Label 5897 2765 1    44   ~ 0
+Text Label 5710 2750 1    44   ~ 0
 BNDIR
-Text Label 7305 2586 1    44   ~ 0
-BP
 Text Label 5650 2750 1    44   ~ 0
 BPDIR
@@
 Text Label 3550 1600 1    44   ~ 0
 DATA_P
-Text Label 7241 2586 1    44   ~ 0
-N$29
 Text Label 4586 5210 0    44   ~ 0
 Standby
@@
 $EndComp
 $Comp
-L +3.3V P+19
-U 1 1 520EEF40
-P 7850 4350
-F 0 "P+19" V 7850 4350 50  0001 L BNN
-F 1 "+3.3V" V 7900 4350 30  0000 L BNN
-F 2 "" H 7850 4350 60  0000 C CNN
-F 3 "" H 7850 4350 60  0000 C CNN
-	1    7850 4350
-	1    0    0    1
-$EndComp
-$Comp
 L GND SUPPLY22
 U 1 1 520EEF6D
@@
 Wire Wire Line
 	5950 4200 5950 4500
-Wire Wire Line
-	7850 3950 7850 4300
-Wire Wire Line
-	8450 3600 8400 3600
-Wire Wire Line
-	8450 3600 8450 4250
 Connection ~ 3450 6000
 Wire Wire Line
@@
 Connection ~ 1400 3000
 Wire Wire Line
-	8150 2500 8500 2500
-Wire Wire Line
-	8500 3500 8400 3500
-Wire Wire Line
-	8500 2500 8500 3500
+	8150 2500 8450 2500
+Wire Wire Line
+	8400 3500 8500 3500
+Wire Wire Line
+	8450 2500 8450 4250
 Connection ~ 8150 2500
-Connection ~ 8500 3500
+Connection ~ 8450 3500
 Wire Wire Line
 	4600 4100 4850 4100
@@
 	7950 2700 7950 2750
 Wire Wire Line
-	8650 2700 8650 4050
+	8650 4050 8650 2700
 Wire Wire Line
 	8650 3400 8400 3400
@@
 Connection ~ 8250 2500
 Wire Wire Line
-	7100 2700 8650 2700
+	8650 2700 7100 2700
 Connection ~ 8250 2700
 Wire Wire Line
-	7850 4150 8300 4150
-Wire Wire Line
-	8300 4150 8300 4250
-Connection ~ 7850 4150
-Wire Wire Line
-	8650 4050 7650 4050
-Wire Wire Line
-	8350 4050 8350 4250
-Connection ~ 8350 4050
+	8300 4000 8300 4250
+Wire Wire Line
+	7650 4050 8650 4050
 Wire Wire Line
 	8150 3950 8150 4000
 Wire Wire Line
-	8150 4000 8400 4000
-Wire Wire Line
-	8400 4000 8400 4250
+	8400 4250 8400 4050
+Connection ~ 8400 4050
+Wire Wire Line
+	8150 4000 8300 4000
+Wire Wire Line
+	8400 3600 8400 3950
+Wire Wire Line
+	8400 3950 8350 3950
+Wire Wire Line
+	8350 3950 8350 4250
+Wire Wire Line
+	7850 3950 7850 4150
+Wire Wire Line
+	7850 4150 8450 4150
+Connection ~ 8450 4150
+NoConn ~ 5900 3500
+NoConn ~ 5950 3500
 $EndSCHEMATC

Commit message: Changed resistors and capacitors from 0402 to 0603 package
Parts:
- renumbered C2 to C1, C16 to C10, C10 to C11, C17 to C12, C6 to C13, C27 to C14, C7 to C15, C28 to C16, C29 to C17, C12 to C2, C30 to C21, C8 to C22, C31 to C23, C9 to C24, C21 to C25, C25 to C26, C22 to C27, C23 to C28, C24 to C29, C13 to C3, C26 to C30, C14 to C4, C3 to C5, C4 to C6, C5 to C7, C1 to C8, C15 to C9, CMT821 to CMT1, D6 to D2, D2 to D3, D3 to D5, D5 to D6, IC5 to IC3, IC3 to IC4, IC4 to IC5, J4 to J2, JP3 to JP1, JP4 to JP2, JP2 to JP3, JP1 to JP4, MPU91501 to MPU1, P+9 to P+10, P+15 to P+14, P+16 to P+15, P+17 to P+16, P+18 to P+17, P+20 to P+18, P+22 to P+9, R17 to R1, R5 to R10, R13 to R11, R14 to R12, R15 to R13, R6 to R14, R7 to R15, R11 to R16, R18 to R2, R8 to R3, R9 to R4, R16 to R5, R2 to R6, R4 to R7, R1 to R8, R3 to R9, SUPPLY11 to SUPPLY10, SUPPLY12 to SUPPLY11, SUPPLY8 to SUPPLY12, SUPPLY15 to SUPPLY14, SUPPLY16 to SUPPLY15, SUPPLY18 to SUPPLY16, SUPPLY19 to SUPPLY18, SUPPLY22 to SUPPLY19, SUPPLY9 to SUPPLY8, SUPPLY10 to SUPPLY9, ??1 to U1, U1 to U2

Commit message: Modified part labels added modules
Parts:
- R14: value ?M -> 150R
- R15: value ?M -> 100R
- renumbered U1 to B1, IC4 to IC3, IC5 to IC4, MPU1 to S1, IC3 to S2
Changed lines of the file:
@@
 U 1 1 520F18EE
 P 8000 4850
-F 0 "D3" H 8000 4850 30  0000 C CNN
-F 1 "SMAJ5.0A" H 7950 4850 30  0000 C CNN
+F 0 "D3" H 8000 4800 30  0000 C CNN
+F 1 "SMAJ5.0A" H 8000 4750 30  0000 C CNN
 F 2 "" H 8000 4850 30  0001 C CNN
 F 3 "" H 8000 4850 30  0001 C CNN
@@
 U 1 1 520F18ED
 P 8100 4850
-F 0 "D5" H 8100 4850 30  0000 C CNN
-F 1 "SMAJ5.0A" H 8050 4850 30  0000 C CNN
+F 0 "D5" H 8100 4800 30  0000 C CNN
+F 1 "SMAJ5.0A" H 8100 4900 30  0000 C CNN
 F 2 "" H 8100 4850 30  0001 C CNN
 F 3 "" H 8100 4850 30  0001 C CNN
@@
 U 1 1 520F18EC
 P 8000 5250
-F 0 "D4" H 8000 5250 30  0000 C CNN
-F 1 "SMAJ5.0A" H 7950 5250 30  0000 C CNN
+F 0 "D4" H 8000 5200 30  0000 C CNN
+F 1 "SMAJ5.0A" H 8000 5150 30  0000 C CNN
 F 2 "" H 8000 5250 30  0001 C CNN
 F 3 "" H 8000 5250 30  0001 C CNN
@@
 U 1 1 520F18EB
 P 8100 5250
-F 0 "D6" H 8100 5250 30  0000 C CNN
-F 1 "SMAJ5.0A" H 8050 5250 30  0000 C CNN
+F 0 "D6" H 8100 5200 30  0000 C CNN
+F 1 "SMAJ5.0A" H 8100 5300 30  0000 C CNN
 F 2 "" H 8100 5250 30  0001 C CNN
 F 3 "" H 8100 5250 30  0001 C CNN
@@
 U 1 1 520F18E7
 P 7850 4850
-F 0 "D2" H 7850 4850 30  0000 C CNN
-F 1 "SMAJ5.0A" H 7800 4850 30  0000 C CNN
+F 0 "D2" H 7850 4800 30  0000 C CNN
+F 1 "SMAJ5.0A" H 7850 4750 30  0000 C CNN
 F 2 "" H 7850 4850 30  0001 C CNN
 F 3 "" H 7850 4850 30  0001 C CNN
@@
 $EndComp
 $Comp
-L IC_SN74LVC1T45 IC4
+L IC_SN74LVC1T45 IC3
 U 1 1 520F18C1
 P 4900 1650
-F 0 "IC4" H 4700 1750 30  0000 C CNN
+F 0 "IC3" H 4700 1750 30  0000 C CNN
 F 1 "SN74LVC1T45DCKR" H 5050 1500 30  0000 C CNN
 F 2 "" H 4900 1650 30  0001 C CNN
@@
 $EndComp
 $Comp
-L IC_SN74LVC1T45 IC5
+L IC_SN74LVC1T45 IC4
 U 1 1 520F18C0
 P 4900 1900
-F 0 "IC5" H 4700 2000 30  0000 C CNN
+F 0 "IC4" H 4700 2000 30  0000 C CNN
 F 1 "SN74LVC1T45DCKR" H 5050 1750 30  0000 C CNN
 F 2 "" H 4900 1900 30  0001 C CNN
@@
 $EndComp
 $Comp
-L IC_MT9V032 IC3
+L IC_MT9V032 S2
 U 1 1 520F18BF
 P 2600 3850
-F 0 "IC3" H 2000 4400 30  0000 C CNN
+F 0 "S2" H 2000 4400 30  0000 C CNN
 F 1 "MT9V032" H 2000 4350 30  0000 C CNN
 F 2 "" H 2600 3850 30  0001 C CNN
@@
 $EndComp
 $Comp
-L R_R R7
-U 1 1 520F18D5
-P 4050 1850
-F 0 "R7" H 4100 1850 30  0000 C CNN
-F 1 "0R" H 3950 1850 30  0000 C CNN
-F 2 "" H 4050 1850 30  0001 C CNN
-F 3 "" H 4050 1850 30  0001 C CNN
-	1    4050 1850
-	1    0    0    -1
-$EndComp
-$Comp
 L R_R R10
 U 1 1 520F18D4
@@
 U 1 1 520F18D1
 P 8600 4750
-F 0 "R16" H 8650 4750 30  0000 C CNN
-F 1 "1M" H 8500 4750 30  0000 C CNN
+F 0 "R16" H 8750 4750 30  0000 C CNN
+F 1 "1M" H 8750 4700 30  0000 C CNN
 F 2 "" H 8600 4750 30  0001 C CNN
 F 3 "" H 8600 4750 30  0001 C CNN
@@
 U 1 1 51F9DBB2
 P 7500 5350
-F 0 "R15" H 7550 5350 30  0000 C CNN
-F 1 "?M" H 7450 5350 30  0000 C CNN
+F 0 "R15" H 7650 5400 30  0000 C CNN
+F 1 "100R" H 7500 5400 30  0000 C CNN
 F 2 "" H 7500 5350 30  0001 C CNN
 F 3 "" H 7500 5350 30  0001 C CNN
@@
 U 1 1 51F9DBBD
 P 7300 5350
-F 0 "R14" H 7350 5350 30  0000 C CNN
-F 1 "?M" H 7250 5350 30  0000 C CNN
+F 0 "R14" H 7350 5400 30  0000 C CNN
+F 1 "150R" H 7200 5400 30  0000 C CNN
 F 2 "" H 7300 5350 30  0001 C CNN
 F 3 "" H 7300 5350 30  0001 C CNN
@@
 $EndComp
 $Comp
-L MPU-9150 MPU1
+L MPU-9150 S1
 U 1 1 520FDEB8
 P 7900 3350
-F 0 "MPU1" H 7900 3350 60  0000 C CNN
+F 0 "S1" H 7900 3350 60  0000 C CNN
 F 1 "MPU-9150" H 7950 3250 60  0001 C CNN
 F 2 "" H 7900 3350 60  0000 C CNN
@@
 $EndComp
 $Comp
-L BEAD U1
+L BEAD B1
 U 1 1 5211703C
 P 4250 2950
-F 0 "U1" H 4350 3000 60  0000 C CNN
+F 0 "B1" H 4350 3000 60  0000 C CNN
 F 1 "BEAD" H 4400 3100 60  0000 C CNN
 F 2 "" H 4250 2950 60  0000 C CNN
@@
 NoConn ~ 5900 3500
 NoConn ~ 5950 3500
+$Comp
+L R_R R7
+U 1 1 520F18D5
+P 4050 1850
+F 0 "R7" H 4100 1850 30  0000 C CNN
+F 1 "0R" H 3950 1850 30  0000 C CNN
+F 2 "" H 4050 1850 30  0001 C CNN
+F 3 "" H 4050 1850 30  0001 C CNN
+	1    4050 1850
+	1    0    0    -1
+$EndComp
 $EndSCHEMATC

Commit message: Added stacked usb and removed micro usb Added logic translator for spi rather than i2c master
Parts:
- removed JP2: JP2Q, jumper-JP2Q, symbol JP2Q
- removed SATA_PRIMARY1: 67800-5005, symbol J_SATA7
- removed SUPPLY7: GND, symbol GND
- added IC?: SN74LVC1T45DCKR, symbol IC_SN74LVC1T45
- added JP?: JP_JP1Q, jumper-JP1, symbol JP_JP1Q
- added P+?: +5V, symbol +5V
- added R?: 10K, symbol R_R
- added R?: 0R, symbol R_R
- added SUPPLY?: GND, symbol GND
- added U?: GSB311231HR, USB Stacked, symbol GSB311231HR
- USB1: value MOLEX-47346-0001 -> WM1399CT-ND
- renumbered BLUE_LED1 to L1, GREEN_LED1 to L2, RED_LED1 to L3
Connections:
- net labels removed: DATA_N, DATA_P
- wire segments 434 -> 445

Commit message: Added stacked usb
Parts:
- removed JP5: JP_JP1Q, jumper-JP1, symbol JP_JP1Q
- removed R10: 1K, symbol R_R
- removed SATA_SLAVE_EXT1: 67800-5005, symbol J_SATA7
- removed SUPPLY4: GND, symbol GND
- removed USB1: WM1399CT-ND, symbol USB_MOLEX-47346-0001
- added P+?: +5V, symbol +5V
- added R?: 1K, symbol R_R
- added SUPPLY?: GND, symbol GND
Connections:
- net labels removed: BNDIR, BPDIR
- wire segments 445 -> 446
- no-connect marks 11 -> 7

Commit message: Added current detector for externally powered device Added MOSFET to enable/disable power to external device
Parts:
- removed P+?: +5V, symbol +5V
- added P+?: +3.3V, symbol +3.3V
- added Q?: MOSFET, symbol MOSFET
- added R?: ?, symbol R_R
- added SUPPLY?: GND, symbol GND
- added U?: MAX4372, symbol MAX4372
Connections:
- wire segments 446 -> 453
Other:
- moved on the sheet: B1, C1, C14, C21, C5, FB1, FB2, L1, U?
