File: kicad/stereo-camera-board.sch (KiCad schematic (older format))
At the start: 123 parts, among them IC1 ZLDO1117G33TA, IC2 MCP1700T-2502E/TT, IC3 SN74LVC1T45DCKR, IC4 SN74LVC1T45DCKR, J2 DIGILENT-JTAG, U2 ATXMEGA256A3-AU

Commit message: Removed load detection Added simple transistor to provide power to external circuit Added diode to prevent power from secondary usb
Parts:
- removed P+?: +3.3V, symbol +3.3V
- removed Q?: MOSFET, symbol MOSFET
- removed R?: ?, symbol R_R
- removed SUPPLY?: GND, symbol GND
- removed U?: MAX4372, symbol MAX4372
- added D?: SMAJ5.0A, symbol D_D-ZENER
- added JP?: JP_JP1Q, jumper-JP1, symbol JP_JP1Q
- added R?: 1K, symbol R_R
- added SUPPLY?: GND, symbol GND
- added T?: -NPN-SOT23-EBC, transistor-SOT23-EBC, symbol -NPN-SOT23-EBC
Connections:
- wire segments 453 -> 455

Commit message: Added transistors to materials.txt Added transistors with biasing resistors to stereo-camera-board.sch Updated pdf
Parts:
- removed R?: 1K, symbol R_R
- removed SUPPLY?: GND, symbol GND
- added D?: SMAJ5.0A, symbol D_D-ZENER
- added P+?: +5V, symbol +5V
- added R? (x2): ?, symbol R_R
- added T?: -NPN-SOT23-EBC, transistor-SOT23-EBC, symbol -NPN-SOT23-EBC
Connections:
- wire segments 455 -> 460

Commit message: Added transistors for controlling slave board signal Added transistor for slave board loopback
Parts:
- removed D?: SMAJ5.0A, symbol D_D-ZENER
- removed P+?: +5V, symbol +5V
- removed R?: ?, symbol R_R
- removed T?: -NPN-SOT23-EBC, transistor-SOT23-EBC, symbol -NPN-SOT23-EBC
- added R?: 10K, symbol R_R
- added R?: 900R, symbol R_R
- added R?: 10k, symbol R_R
- added R?: ?, symbol R_R
- added SUPPLY?: GND, symbol GND
- added T?: 2N2907A, transistor-TO18, symbol 2N2907A-PNP-TO18-EBC
- added T? (x3): -NPN-SOT23-EBC, transistor-SOT23-EBC, symbol -NPN-SOT23-EBC
Connections:
- wire segments 460 -> 457
Changed lines of the file:
@@
-$EndComp
-$Comp
-L -NPN-SOT23-EBC T?
-U 1 1 52EC9FFB
-P 2500 650
-F 0 "T?" H 2100 950 50  0000 L BNN
-F 1 "-NPN-SOT23-EBC" H 2100 850 50  0000 L BNN
-F 2 "transistor-SOT23-EBC" H 2500 800 50  0001 C CNN
-F 3 "P2N2222A" H 2500 650 60  0000 C CNN
-	1    2500 650
-	0    1    1    0
 $EndComp
 $Comp
@@
 L -NPN-SOT23-EBC T?
 U 1 1 52F46D80
-P 2100 1650
-F 0 "T?" H 1700 1950 50  0000 L BNN
-F 1 "-NPN-SOT23-EBC" V 1700 1850 50  0001 L BNN
-F 2 "transistor-SOT23-EBC" H 2100 1800 50  0001 C CNN
-F 3 "P2N2222A" H 2100 1650 60  0000 C CNN
-	1    2100 1650
+P 1900 1050
+F 0 "T?" H 1800 1100 50  0000 L BNN
+F 1 "-NPN-SOT23-EBC" V 1500 1250 50  0001 L BNN
+F 2 "transistor-SOT23-EBC" H 1900 1200 50  0001 C CNN
+F 3 "P2N2222A" H 1900 1050 60  0000 C CNN
+	1    1900 1050
 	0    1    1    0
 $EndComp
 $Comp
-L D_D-ZENER D?
-U 1 1 52F47019
-P 2300 1550
-F 0 "D?" H 2300 1500 30  0000 C CNN
-F 1 "SMAJ5.0A" H 2300 1600 30  0000 C CNN
-F 2 "" H 2300 1550 30  0001 C CNN
-F 3 "" H 2300 1550 30  0001 C CNN
-	1    2300 1550
+L R_R R?
+U 1 1 52F482F6
+P 2200 550
+F 0 "R?" H 2200 600 30  0000 C CNN
+F 1 "?" H 2200 500 30  0000 C CNN
+F 2 "" H 2200 550 30  0001 C CNN
+F 3 "" H 2200 550 30  0001 C CNN
+	1    2200 550
+	1    0    0    -1
+$EndComp
+$Comp
+L 2N2907A-PNP-TO18-EBC T?
+U 1 1 52F70F9A
+P 2500 650
+F 0 "T?" H 2400 700 50  0000 L BNN
+F 1 "2N2907A" H 2400 550 50  0000 L BNN
+F 2 "transistor-TO18" H 2500 800 50  0001 C CNN
+F 3 "" H 2500 650 60  0000 C CNN
+	1    2500 650
 	0    1    1    0
 $EndComp
-Wire Wire Line
-	2300 1600 2300 1750
+$Comp
+L GND SUPPLY?
+U 1 1 52F71BCA
+P 1600 1200
+F 0 "SUPPLY?" H 1600 1200 30  0001 L BNN
+F 1 "GND" H 1552 1120 30  0000 L BNN
+F 2 "" H 1600 1200 60  0000 C CNN
+F 3 "" H 1600 1200 60  0000 C CNN
+	1    1600 1200
+	1    0    0    -1
+$EndComp
+$Comp
+L R_R R?
+U 1 1 52F71BD0
+P 1700 1050
+F 0 "R?" H 1650 1000 30  0000 C CNN
+F 1 "10K" H 1650 1100 30  0000 C CNN
+F 2 "" H 1700 1050 30  0001 C CNN
+F 3 "" H 1700 1050 30  0001 C CNN
+	1    1700 1050
+	0    -1   -1   0
+$EndComp
+$Comp
+L R_R R?
+U 1 1 52F71E2E
+P 1600 950
+F 0 "R?" H 1600 900 30  0000 C CNN
+F 1 "900R" H 1600 1000 30  0000 C CNN
+F 2 "" H 1600 950 30  0001 C CNN
+F 3 "" H 1600 950 30  0001 C CNN
+	1    1600 950
+	-1   0    0    1
+$EndComp
+$Comp
+L R_R R?
+U 1 1 52F722E6
+P 2700 650
+F 0 "R?" H 2700 700 30  0000 C CNN
+F 1 "10k" H 2700 600 30  0000 C CNN
+F 2 "" H 2700 650 30  0001 C CNN
+F 3 "" H 2700 650 30  0001 C CNN
+	1    2700 650
+	0    -1   -1   0
+$EndComp
+$Comp
+L -NPN-SOT23-EBC T?
+U 1 1 52F72812
+P 5700 600
+F 0 "T?" H 5600 650 50  0000 L BNN
+F 1 "-NPN-SOT23-EBC" V 5600 300 50  0000 L BNN
+F 2 "transistor-SOT23-EBC" H 5700 750 50  0001 C CNN
+F 3 "" H 5700 600 60  0000 C CNN
+	1    5700 600
+	0    1    1    0
+$EndComp
+$Comp
+L -NPN-SOT23-EBC T?
+U 1 1 52F8E804
+P 9750 950
+F 0 "T?" H 9650 1000 50  0000 L BNN
+F 1 "-NPN-SOT23-EBC" V 9650 650 50  0000 L BNN
+F 2 "transistor-SOT23-EBC" H 9750 1100 50  0001 C CNN
+F 3 "" H 9750 950 60  0000 C CNN
+	1    9750 950
+	0    1    1    0
+$EndComp
+$Comp
+L -NPN-SOT23-EBC T?
+U 1 1 52F8E814
+P 9750 1300
+F 0 "T?" H 9650 1350 50  0000 L BNN
+F 1 "-NPN-SOT23-EBC" V 9650 1000 50  0000 L BNN
+F 2 "transistor-SOT23-EBC" H 9750 1450 50  0001 C CNN
+F 3 "" H 9750 1300 60  0000 C CNN
+	1    9750 1300
+	0    1    1    0
+$EndComp
+$Comp
+L R_R R?
+U 1 1 52F8EA71
+P 5900 600
+F 0 "R?" H 5950 600 30  0000 C CNN
+F 1 "?" V 5800 600 30  0000 C CNN
+F 2 "" H 5900 600 30  0001 C CNN
+F 3 "" H 5900 600 30  0001 C CNN
+	1    5900 600
+	0    -1   -1   0
+$EndComp
 Connection ~ 2300 1350
 Wire Wire Line
-	2300 1050 2300 1500
-Wire Wire Line
 	2300 750  2300 950
-Wire Wire Line
-	1700 550  1700 2150
-Wire Wire Line
-	2300 1350 2800 1350
 Wire Wire Line
 	3100 1350 4500 1350
@@
 Connection ~ 2850 750
 Wire Wire Line
-	1900 1750 1900 1650
-$Comp
-L +5V P+?
-U 1 1 52F48098
-P 1900 1600
-F 0 "P+?" V 1900 1600 50  0001 L BNN
-F 1 "+5V" V 1950 1600 30  0000 L BNN
-F 2 "" H 1900 1600 60  0000 C CNN
-F 3 "" H 1900 1600 60  0000 C CNN
-	1    1900 1600
-	1    0    0    -1
-$EndComp
-Wire Wire Line
-	2100 1550 2100 1350
-Wire Wire Line
-	1750 1350 1750 2150
-$Comp
-L R_R R?
-U 1 1 52F482F6
-P 2100 550
-F 0 "R?" H 2150 550 30  0000 C CNN
-F 1 "?" H 2050 550 30  0000 C CNN
-F 2 "" H 2100 550 30  0001 C CNN
-F 3 "" H 2100 550 30  0001 C CNN
-	1    2100 550
-	1    0    0    -1
-$EndComp
-Wire Wire Line
-	2000 550  1700 550
-Wire Wire Line
-	2200 550  2500 550
-$Comp
-L R_R R?
-U 1 1 52F487AA
-P 1900 1350
-F 0 "R?" H 1950 1350 30  0000 C CNN
-F 1 "?" H 1850 1350 30  0000 C CNN
-F 2 "" H 1900 1350 30  0001 C CNN
-F 3 "" H 1900 1350 30  0001 C CNN
-	1    1900 1350
-	1    0    0    -1
-$EndComp
-Wire Wire Line
-	1750 1350 1800 1350
-Wire Wire Line
-	2100 1350 2000 1350
+	2300 1350 2800 1350
+Wire Wire Line
+	2300 550  2700 550
+Wire Wire Line
+	2100 550  2100 1150
+Wire Wire Line
+	1700 1150 1600 1150
+Connection ~ 1700 1150
+Wire Wire Line
+	1900 950  1700 950
+Connection ~ 1700 950
+Wire Wire Line
+	1500 950  1500 2050
+Connection ~ 2500 550
+Wire Wire Line
+	2300 1050 2300 1350
+Wire Wire Line
+	5700 500  5900 500
 $EndSCHEMATC

Commit message: Put micro usb port back Updated pdf
Parts:
- removed JP?: JP_JP1Q, jumper-JP1, symbol JP_JP1Q
- removed T? (x2): -NPN-SOT23-EBC, transistor-SOT23-EBC, symbol -NPN-SOT23-EBC
- added C?: 4.7nf, symbol C_C
- added D? (x2): SMAJ5.0A, symbol D_D-ZENER
- added P+?: +5V, symbol +5V
- added R?: 1M, symbol R_R
- added SUPPLY?: GND, symbol GND
- added USB?: USB_MOLEX-47346-0001, usb_con-update-MOLEX-47364-0001, symbol USB_MOLEX-47346-0001
- R?: value ? -> 1K
- R?: value 10K -> 22K
- R?: value 900R -> 2.2K
Connections:
- wire segments 457 -> 461

Commit message: Added esd protection ic
Parts:
- removed D2, D3, D4, D5, D6: SMAJ5.0A, symbol D_D-ZENER
- added U?: MAX3207E, symbol MAX3207E
Connections:
- wire segments 461 -> 459
Changed lines of the file:
@@
-$EndComp
-$Comp
-L D_D-ZENER D3
-U 1 1 520F18EE
-P 10100 5900
-F 0 "D3" H 10100 5850 30  0000 C CNN
-F 1 "SMAJ5.0A" H 10100 5800 30  0000 C CNN
-F 2 "" H 10100 5900 30  0001 C CNN
-F 3 "" H 10100 5900 30  0001 C CNN
-	1    10100 5900
-	0    -1   -1   0
-$EndComp
-$Comp
-L D_D-ZENER D5
-U 1 1 520F18ED
-P 10000 5900
-F 0 "D5" H 10000 5850 30  0000 C CNN
-F 1 "SMAJ5.0A" H 10000 5950 30  0000 C CNN
-F 2 "" H 10000 5900 30  0001 C CNN
-F 3 "" H 10000 5900 30  0001 C CNN
-	1    10000 5900
-	0    -1   -1   0
-$EndComp
-$Comp
-L D_D-ZENER D4
-U 1 1 520F18EC
-P 10100 5600
-F 0 "D4" H 10100 5550 30  0000 C CNN
-F 1 "SMAJ5.0A" H 10100 5500 30  0000 C CNN
-F 2 "" H 10100 5600 30  0001 C CNN
-F 3 "" H 10100 5600 30  0001 C CNN
-	1    10100 5600
-	0    -1   -1   0
-$EndComp
-$Comp
-L D_D-ZENER D6
-U 1 1 520F18EB
-P 10000 5600
-F 0 "D6" H 10000 5550 30  0000 C CNN
-F 1 "SMAJ5.0A" H 10000 5650 30  0000 C CNN
-F 2 "" H 10000 5600 30  0001 C CNN
-F 3 "" H 10000 5600 30  0001 C CNN
-	1    10000 5600
-	0    -1   -1   0
-$EndComp
-$Comp
-L D_D-ZENER D2
-U 1 1 520F18E7
-P 10250 5900
-F 0 "D2" H 10250 5850 30  0000 C CNN
-F 1 "SMAJ5.0A" H 10250 5800 30  0000 C CNN
-F 2 "" H 10250 5900 30  0001 C CNN
-F 3 "" H 10250 5900 30  0001 C CNN
-	1    10250 5900
-	0    -1   -1   0
 $EndComp
 $Comp
@@
 L D_D-ZENER D?
 U 1 1 52F991C9
-P 9850 5400
-F 0 "D?" H 9850 5350 30  0000 C CNN
-F 1 "SMAJ5.0A" H 9850 5450 30  0000 C CNN
-F 2 "" H 9850 5400 30  0001 C CNN
-F 3 "" H 9850 5400 30  0001 C CNN
-	1    9850 5400
+P 8850 6150
+F 0 "D?" H 8850 6100 30  0000 C CNN
+F 1 "SMAJ5.0A" H 8850 6200 30  0000 C CNN
+F 2 "" H 8850 6150 30  0001 C CNN
+F 3 "" H 8850 6150 30  0001 C CNN
+	1    8850 6150
 	0    -1   -1   0
 $EndComp
@@
 L +5V P+?
 U 1 1 52F996AF
-P 9850 5250
-F 0 "P+?" V 9850 5250 50  0001 L BNN
-F 1 "+5V" V 9900 5250 30  0000 L BNN
-F 2 "" H 9850 5250 60  0000 C CNN
-F 3 "" H 9850 5250 60  0000 C CNN
-	1    9850 5250
+P 8850 6000
+F 0 "P+?" V 8850 6000 50  0001 L BNN
+F 1 "+5V" V 8900 6000 30  0000 L BNN
+F 2 "" H 8850 6000 60  0000 C CNN
+F 3 "" H 8850 6000 60  0000 C CNN
+	1    8850 6000
 	1    0    0    -1
 $EndComp
@@
 	0    -1   -1   0
 $EndComp
+$Comp
+L C_C C30
+U 1 1 520F18F0
+P 4050 1950
+F 0 "C30" V 4100 1800 30  0000 C CNN
+F 1 "4.7nf" V 4100 2000 30  0000 C CNN
+F 2 "" H 4050 1950 30  0001 C CNN
+F 3 "" H 4050 1950 30  0001 C CNN
+	1    4050 1950
+	0    1    -1   0
+$EndComp
+$Comp
+L MAX3207E U?
+U 1 1 52FB9656
+P 9500 6250
+F 0 "U?" H 9350 6550 60  0000 C CNN
+F 1 "MAX3207E" H 9500 6650 60  0000 C CNN
+F 2 "" H 9500 6250 60  0000 C CNN
+F 3 "" H 9500 6250 60  0000 C CNN
+	1    9500 6250
+	-1   0    0    1
+$EndComp
 Wire Wire Line
 	2300 750  2300 950
@@
 Connection ~ 4850 700
 Connection ~ 4850 800
-Wire Wire Line
-	10000 5500 10000 5550
-Wire Wire Line
-	10100 5500 10100 5550
-Wire Wire Line
-	8950 5500 10350 5500
-Connection ~ 10000 5500
-Connection ~ 10250 5500
-Connection ~ 10100 5500
 Wire Wire Line
 	6650 3050 8250 3050
@@
 	7400 4650 5900 4650
 Wire Wire Line
-	10000 5650 10000 5850
-Connection ~ 10000 5750
-Wire Wire Line
-	10100 5650 10100 5850
-Connection ~ 10100 5800
-Wire Wire Line
 	10450 3100 10750 3100
 Wire Wire Line
@@
 Wire Wire Line
 	3350 2300 3500 2300
-Wire Wire Line
-	10100 5950 10100 6300
-Wire Wire Line
-	10000 6000 10000 5950
-Connection ~ 10100 6000
-Connection ~ 10000 6000
 Wire Wire Line
 	8200 4700 8200 4100
@@
 	4100 1850 3950 1850
 Connection ~ 3950 1950
-Wire Wire Line
-	10000 6000 10300 6000
 Connection ~ 4150 2050
 Wire Wire Line
@@
 Wire Wire Line
 	2850 800  2900 800
-Connection ~ 10250 6000
 Wire Wire Line
 	2850 750  2700 750
@@
 Wire Wire Line
 	5700 500  5900 500
-Wire Wire Line
-	10350 5500 10350 5700
-Wire Wire Line
-	10250 5500 10250 5850
 Connection ~ 10100 6150
-Wire Wire Line
-	10250 6000 10250 5950
 Wire Wire Line
 	10250 6300 10300 6300
@@
 	8900 4100 8900 5800
 Wire Wire Line
-	9850 5300 9850 5350
-Wire Wire Line
-	9850 5450 9850 5500
-Wire Wire Line
-	8950 5500 8950 5450
-Connection ~ 9850 5500
+	8850 6050 8850 6100
+Wire Wire Line
+	8850 6200 8850 6250
+Wire Wire Line
+	8950 5450 8950 6250
 Wire Wire Line
 	5950 1550 5950 1450
@@
 Wire Wire Line
 	4100 1950 4150 1950
-$Comp
-L C_C C30
-U 1 1 520F18F0
-P 4050 1950
-F 0 "C30" V 4100 1800 30  0000 C CNN
-F 1 "4.7nf" V 4100 2000 30  0000 C CNN
-F 2 "" H 4050 1950 30  0001 C CNN
-F 3 "" H 4050 1950 30  0001 C CNN
-	1    4050 1950
-	0    1    -1   0
-$EndComp
 Wire Wire Line
 	4150 1650 4150 2050
+Wire Wire Line
+	9100 6050 9100 5800
+Connection ~ 9100 5800
+Wire Wire Line
+	10100 6150 9900 6150
+Wire Wire Line
+	9900 6150 9900 6250
+Wire Wire Line
+	9950 5750 9950 6450
+Wire Wire Line
+	9950 6450 9900 6450
+Connection ~ 9950 5750
+Wire Wire Line
+	8850 6250 9100 6250
+Connection ~ 8950 6250
+Wire Wire Line
+	10100 6000 10100 6300
+Wire Wire Line
+	10300 6000 10100 6000
+Wire Wire Line
+	10350 5700 8950 5700
+Connection ~ 8950 5700
 $EndSCHEMATC

Commit message: Tied down all remaining signals Removed jtag
Parts:
- removed D?: SMAJ5.0A, symbol D_D-ZENER
- removed J2: DIGILENT-JTAG, symbol J_DIGILENT-JTAG
- removed JP3: ~, symbol JP_PINHD-2X3
- removed P+13, P+15: +3.3V, symbol +3.3V
- removed R?: ?, symbol R_R
- removed SUPPLY14, SUPPLY8, SUPPLY?: GND, symbol GND
- removed T?: -NPN-SOT23-EBC, transistor-SOT23-EBC, symbol -NPN-SOT23-EBC
- added JP?: JP_JP1Q, jumper-JP1, symbol JP_JP1Q
- added R?: 100K, symbol R_R
- added SUPPLY?: GND, symbol GND
- R6: value 100R -> 0R
- R7, R?: value 0R -> 100R
Connections:
- wire segments 459 -> 449

Commit message: Added jumpers for remaining pins
Parts:
- added JP? (x2): JP2E, jumper-JP2, symbol JP2E
Connections:
- wire segments 449 -> 462
Changed lines of the file:
@@
 	7250 1000 8450 1000
 Wire Wire Line
-	7850 4100 7850 5550
-Wire Wire Line
-	7900 5550 7900 4100
-Wire Wire Line
-	7950 4400 7950 5550
+	7850 4100 7850 5600
+Wire Wire Line
+	7900 4100 7900 5650
+Wire Wire Line
+	7950 4400 7950 5700
 Wire Wire Line
 	8000 4400 7950 4400
@@
 Wire Wire Line
 	1550 6300 8000 6300
+$Comp
+L JP2E JP?
+U 1 1 530D6E52
+P 7600 5900
+F 0 "JP?" V 7415 5900 50  0000 L BNN
+F 1 "JP2E" V 7790 5900 50  0000 L BNN
+F 2 "jumper-JP2" H 7600 6050 50  0001 C CNN
+F 3 "" H 7600 5900 60  0000 C CNN
+	1    7600 5900
+	-1   0    0    1
+$EndComp
+Wire Wire Line
+	7850 5600 7500 5600
+Wire Wire Line
+	7500 5600 7500 5800
+Wire Wire Line
+	7900 5650 7600 5650
+Wire Wire Line
+	7600 5650 7600 5800
+Wire Wire Line
+	7950 5700 7700 5700
+Wire Wire Line
+	7700 5700 7700 5800
+$Comp
+L JP2E JP?
+U 1 1 530D753E
+P 8700 1900
+F 0 "JP?" V 8515 1900 50  0000 L BNN
+F 1 "JP2E" V 8890 1900 50  0000 L BNN
+F 2 "jumper-JP2" H 8700 2050 50  0001 C CNN
+F 3 "" H 8700 1900 60  0000 C CNN
+	1    8700 1900
+	1    0    0    -1
+$EndComp
+Wire Wire Line
+	8600 3400 8600 2000
+Wire Wire Line
+	8650 2050 8650 3400
+Wire Wire Line
+	8650 2050 8700 2050
+Wire Wire Line
+	8700 2050 8700 2000
+Wire Wire Line
+	8700 3400 8700 2100
+Wire Wire Line
+	8700 2100 8800 2100
+Wire Wire Line
+	8800 2100 8800 2000
 $EndSCHEMATC

Commit message: Cleaned up some ERC errors More ERC errors left to fix
Parts:
- removed SUPPLY?: GND, symbol GND
- added SUPPLY8: GND, symbol GND
- gave numbers to parts that had none: 27
Connections:
- wire segments 462 -> 465
- no-connect marks 7 -> 10
