File: kicad/stereo-camera-board.kicad_pcb (KiCad board)
At the start: 4 copper layers, 57 x 70 mm, 150 parts, among them IC1 ZLDO1117G33TA, IC2 MCP1700T-2502E/TT, IC3 SN74LVC1T45DCKR, IC4 SN74LVC1T45DCKR, IC5 SN74LVC1T45DCKR, T1 2n2222a, T2 2N2907A, U1 GSB311231HR, U2 ATXMEGA256A3-AU, U3 MAX3207E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

Commit message: Added drill holes for mounting
Parts:
- added Screw4-40: VAL**, ViasAndHoles:Screw4-40, F.Cu at (166.6, 143.9)
- added Screw4-40: VAL**, ViasAndHoles:Screw4-40, F.Cu at (168.7, 82.7)
- added Screw4-40: VAL**, ViasAndHoles:Screw4-40, F.Cu at (124.9, 122.7)
Changed lines of the file:
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@@
 (kicad_pcb (version 3) (host pcbnew "(2014-03-19 BZR 4756)-product")
   (general
-    (links 252)
+    (links 0)
     (no_connects 2)
     (area 107.779144 64.798058 193.061213 155.002)
@@
     (tracks 1183)
     (zones 0)
-    (modules 150)
+    (modules 153)
     (nets 108)
   )
@@
     (mod_text_size 1.5 1.5)
     (mod_text_width 0.15)
-    (pad_size 1.45 1.45)
-    (pad_drill 0.85)
+    (pad_size 3.2639 3.2639)
+    (pad_drill 3.2639)
     (pad_to_mask_clearance 0.2)
     (aux_axis_origin 0 0)
@@
     (pad 1 thru_hole circle (at 0 0) (size 0.3556 0.3556) (drill 0.254) (layers *.Cu))
   )
+  (module ViasAndHoles:Screw4-40 (layer F.Cu)
+    (at 166.55 143.9)
+    (fp_text reference Screw4-40 (at 0 0) (layer F.SilkS)
+      (effects (font (size 1.5 1.5) (thickness 0.15)))
+    )
+    (fp_text value VAL** (at 0 0) (layer F.SilkS)
+      (effects (font (size 1.5 1.5) (thickness 0.15)))
+    )
+    (pad "" np_thru_hole circle (at 0 0) (size 3.2639 3.2639) (drill 3.2639) (layers *.Cu)
+      (clearance 0.006))
+  )
+  (module ViasAndHoles:Screw4-40 (layer F.Cu)
+    (at 168.725 82.7)
+    (fp_text reference Screw4-40 (at 0 0) (layer F.SilkS)
+      (effects (font (size 1.5 1.5) (thickness 0.15)))
+    )
+    (fp_text value VAL** (at 0 0) (layer F.SilkS)
+      (effects (font (size 1.5 1.5) (thickness 0.15)))
+    )
+    (pad "" np_thru_hole circle (at 0 0) (size 3.2639 3.2639) (drill 3.2639) (layers *.Cu)
+      (clearance 0.006))
+  )
+  (module ViasAndHoles:Screw4-40 (layer F.Cu)
+    (at 124.925 122.675)
+    (fp_text reference Screw4-40 (at 0 0) (layer F.SilkS)
+      (effects (font (size 1.5 1.5) (thickness 0.15)))
+    )
+    (fp_text value VAL** (at 0 0) (layer F.SilkS)
+      (effects (font (size 1.5 1.5) (thickness 0.15)))
+    )
+    (pad "" np_thru_hole circle (at 0 0) (size 3.2639 3.2639) (drill 3.2639) (layers *.Cu)
+      (clearance 0.006))
+  )
   (gr_text GND (at 175 84.1) (layer F.SilkS)
